Commit message: clover->drone

File: clover_description/urdf/clover/clover4.xacro (robot description, xacro)
@@ -1,4 +1,4 @@
 <?xml version="1.0"?>
-<robot name="clover" xmlns:xacro="http://ros.org/wiki/xacro">
+<robot name="drone" xmlns:xacro="http://ros.org/wiki/xacro">
   <xacro:arg name="main_camera" default="true"/>
   <xacro:arg name="rangefinder" default="true"/>
@@ -6,6 +6,6 @@
   <xacro:arg name="gps" default="true"/>
   <xacro:arg name="maintain_camera_rate" default="false"/>
-  <xacro:arg name="use_clover_physics" default="false"/>
-  <xacro:include filename="clover4_base.xacro" />
+  <xacro:arg name="use_drone_physics" default="false"/>
+  <xacro:include filename="drone4_base.xacro" />
   <xacro:include filename="../sensors/rpi_cam.urdf.xacro"/>
   <xacro:include filename="../sensors/distance_sensor.urdf.xacro"/>

File: clover_description/urdf/clover/clover4_base.xacro (robot description, xacro)
@@ -1,11 +1,11 @@
 <?xml version="1.0"?>
-<robot name="clover" xmlns:xacro="http://ros.org/wiki/xacro">
+<robot name="drone" xmlns:xacro="http://ros.org/wiki/xacro">
   <xacro:arg name='enable_wind' default='false' />
   <xacro:arg name='enable_logging' default='false' />
-  <xacro:arg name='log_file' default='clover' />
+  <xacro:arg name='log_file' default='drone' />
   <!-- macros for gazebo plugins, sensors -->
   <xacro:include filename="../component_snippets.urdf.xacro" />
   <!-- Instantiate iris "mechanics" -->
-  <xacro:include filename="clover4_physics.xacro" />
+  <xacro:include filename="drone4_physics.xacro" />
   <xacro:if value="$(arg enable_wind)">
     <xacro:wind_plugin_macro
@@ -21,5 +21,5 @@
   </xacro:if>
   <!-- Gazebo plugins -->
-  <xacro:include filename="$(find clover_description)/urdf/clover/clover4_gazebo.xacro" />
+  <xacro:include filename="$(find drone_description)/urdf/drone/drone4_gazebo.xacro" />
   <xacro:if value="$(arg enable_logging)">
     <!-- Instantiate a logger -->

File: clover_description/urdf/clover/clover4_macros.xacro (robot description, xacro)
@@ -17,5 +17,5 @@
 -->
 <!--
-  Clover 4 base model, collision boxes, and other fun stuff. Derived heavily from multirotor_base.xacro
+  Drone 4 base model, collision boxes, and other fun stuff. Derived heavily from multirotor_base.xacro
   from PX4 simulation config files.
 -->
@@ -26,5 +26,5 @@
        Color is not applicable, since the model has textures and is a compound thingy anyway.
   -->
-  <xacro:macro name="clover4_base_macro"
+  <xacro:macro name="drone4_base_macro"
     params="robot_namespace mass body_width body_height *inertia">
     <link name="base_link"></link>
@@ -48,5 +48,5 @@
         <geometry>
           <!-- Note: Texture files are expected to be in the same directory as the model -->
-          <mesh filename="package://clover_description/meshes/clover4/clover_body_solid.dae"
+          <mesh filename="package://drone_description/meshes/drone4/drone_body_solid.dae"
             scale="1 1 1"/>
         </geometry>
@@ -106,5 +106,5 @@
         <origin xyz="0 0 0.025" rpy="0 0 0"/>
         <geometry>
-          <mesh filename="package://clover_description/meshes/clover4/clover_guards_transparent.dae"
+          <mesh filename="package://drone_description/meshes/drone4/drone_guards_transparent.dae"
             scale="1 1 1"/>
         </geometry>
@@ -156,6 +156,6 @@
    </gazebo>
   </xacro:macro>
-  <!-- Rotor joint and link, modified for Clover purposes -->
-  <xacro:macro name="vertical_clover_rotor"
+  <!-- Rotor joint and link, modified for Drone purposes -->
+  <xacro:macro name="vertical_drone_rotor"
     params="robot_namespace suffix direction motor_constant moment_constant parent mass_rotor radius_rotor time_constant_up time_constant_down max_rot_velocity motor_number rotor_drag_coefficient rolling_moment_coefficient mesh *origin *inertia">
     <joint name="rotor_${motor_number}_joint" type="continuous">
@@ -177,5 +177,5 @@
       <visual>
         <geometry>
-          <mesh filename="package://clover_description/meshes/${mesh}"
+          <mesh filename="package://drone_description/meshes/${mesh}"
             scale="1 1 1" />
         </geometry>

File: clover_description/urdf/clover/clover4_physics.xacro (robot description, xacro)
@@ -1,15 +1,15 @@
 <?xml version="1.0"?>
-<!-- Typical physics values for the Clover drone.
+<!-- Typical physics values for the Drone drone.
      NB: Right now the values are wrong, and taken from the 3DR Iris drone description.
      This is subject to change as correct values are calculated.
 -->
-<robot name="clover" xmlns:xacro="http://ros.org/wiki/xacro">
+<robot name="drone" xmlns:xacro="http://ros.org/wiki/xacro">
   <!-- Properties -->
   <xacro:property name="namespace" value="" />
   <xacro:property name="rotor_velocity_slowdown_sim" value="10" />
-  <xacro:if value="$(arg use_clover_physics)">
+  <xacro:if value="$(arg use_drone_physics)">
     <xacro:property name="mass" value="0.7" /> <!-- [kg] -->
   </xacro:if>
-  <xacro:unless value="$(arg use_clover_physics)">
+  <xacro:unless value="$(arg use_drone_physics)">
     <xacro:property name="mass" value="1.5" /> <!-- [kg] -->
   </xacro:unless>
@@ -35,7 +35,7 @@
   <xacro:property name="color" value="DarkGrey" />
   <!-- Property Blocks -->
-  <!-- Clover body inertia -->
+  <!-- Drone body inertia -->
   <!-- Values from CAD program -->
-  <xacro:if value="$(arg use_clover_physics)">
+  <xacro:if value="$(arg use_drone_physics)">
     <xacro:property name="body_inertia">
       <inertia
@@ -47,5 +47,5 @@
   </xacro:if>
   <!-- Box-like inertia -->
-  <xacro:unless value="$(arg use_clover_physics)">
+  <xacro:unless value="$(arg use_drone_physics)">
     <xacro:property name="body_inertia">
       <inertia
@@ -58,5 +58,5 @@
   <!-- inertia of a single rotor -->
   <!-- Values from CAD program -->
-  <xacro:if value="$(arg use_clover_physics)">
+  <xacro:if value="$(arg use_drone_physics)">
     <xacro:property name="rotor_inertia">
       <inertia
@@ -68,5 +68,5 @@
   </xacro:if>
   <!-- Values for a cuboid (cuboid. Height=3mm, width=15mm) -->
-  <xacro:unless value="$(arg use_clover_physics)">
+  <xacro:unless value="$(arg use_drone_physics)">
     <xacro:property name="rotor_inertia">
       <inertia
@@ -78,7 +78,7 @@
   </xacro:unless>
   <!-- Included URDF Files -->
-  <xacro:include filename="clover4_macros.xacro" />
+  <xacro:include filename="drone4_macros.xacro" />
   <!-- Instantiate multirotor_base_macro once -->
-  <xacro:clover4_base_macro
+  <xacro:drone4_base_macro
     robot_namespace="${namespace}"
     mass="${mass}"
@@ -87,7 +87,7 @@
     >
     <xacro:insert_block name="body_inertia" />
-  </xacro:clover4_base_macro>
+  </xacro:drone4_base_macro>
   <!-- Instantiate rotors -->
-  <xacro:vertical_clover_rotor
+  <xacro:vertical_drone_rotor
     robot_namespace="${namespace}"
     suffix="front_right"
@@ -104,9 +104,9 @@
     rotor_drag_coefficient="${rotor_drag_coefficient}"
     rolling_moment_coefficient="${rolling_moment_coefficient}"
-    mesh="clover4/prop_ccw.dae">
+    mesh="drone4/prop_ccw.dae">
     <origin xyz="${arm_length_front_x} -${arm_length_front_y} ${rotor_offset_top}" rpy="0 0 0" />
     <xacro:insert_block name="rotor_inertia" />
-  </xacro:vertical_clover_rotor>
-  <xacro:vertical_clover_rotor
+  </xacro:vertical_drone_rotor>
+  <xacro:vertical_drone_rotor
     robot_namespace="${namespace}"
     suffix="back_left"
@@ -123,9 +123,9 @@
     rotor_drag_coefficient="${rotor_drag_coefficient}"
     rolling_moment_coefficient="${rolling_moment_coefficient}"
-    mesh="clover4/prop_ccw.dae">
+    mesh="drone4/prop_ccw.dae">
     <origin xyz="-${arm_length_back_x} ${arm_length_back_y} ${rotor_offset_top}" rpy="0 0 0" />
     <xacro:insert_block name="rotor_inertia" />
-  </xacro:vertical_clover_rotor>
-  <xacro:vertical_clover_rotor robot_namespace="${namespace}"
+  </xacro:vertical_drone_rotor>
+  <xacro:vertical_drone_rotor robot_namespace="${namespace}"
     suffix="front_left"
     direction="cw"
@@ -141,9 +141,9 @@
     rotor_drag_coefficient="${rotor_drag_coefficient}"
     rolling_moment_coefficient="${rolling_moment_coefficient}"
-    mesh="clover4/prop_cw.dae">
+    mesh="drone4/prop_cw.dae">
     <origin xyz="${arm_length_front_x} ${arm_length_front_y} ${rotor_offset_top}" rpy="0 0 0" />
     <xacro:insert_block name="rotor_inertia" />
-  </xacro:vertical_clover_rotor>
-  <xacro:vertical_clover_rotor robot_namespace="${namespace}"
+  </xacro:vertical_drone_rotor>
+  <xacro:vertical_drone_rotor robot_namespace="${namespace}"
     suffix="back_right"
     direction="cw"
@@ -159,7 +159,7 @@
     rotor_drag_coefficient="${rotor_drag_coefficient}"
     rolling_moment_coefficient="${rolling_moment_coefficient}"
-    mesh="clover4/prop_cw.dae">
+    mesh="drone4/prop_cw.dae">
     <origin xyz="-${arm_length_back_x} -${arm_length_back_y} ${rotor_offset_top}" rpy="0 0 0" />
     <xacro:insert_block name="rotor_inertia" />
-  </xacro:vertical_clover_rotor>
+  </xacro:vertical_drone_rotor>
 </robot>
